File: hardware/no_fly_zone/rev1.0/mcu.kicad_sch (KiCad schematic)
At the start: 23 parts, among them SW1 NRST, SW2 BOOT0, U1 STM32F446RCTx, Y1 8MHz

Commit message: Added quadcopter PCB revision 2 and updated README
Connections:
- net IIS2_IRQ renamed MAG_IRQ
- net TIM2_CH2 renamed TIM5_CH2
- net TIM2_CH3 renamed TIM5_CH3
Changed lines of the file:
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@@
 		)
 	)
-	(hierarchical_label "TIM2_CH3"
+	(hierarchical_label "TIM5_CH3"
 		(shape input)
 		(at 139.7 86.36 0)
@@
 		)
 	)
-	(hierarchical_label "TIM2_CH2"
+	(hierarchical_label "TIM5_CH2"
 		(shape input)
 		(at 139.7 83.82 0)
@@
 		)
 	)
-	(hierarchical_label "IIS2_IRQ"
+	(hierarchical_label "MAG_IRQ"
 		(shape input)
 		(at 139.7 152.4 0)
