File: hardware/no_fly_zone/rev1.0/no_fly_zone.kicad_pcb (KiCad board)
At the start: 4 copper layers, 108.4 x 50 mm, 90 parts, among them J1 ESC, J10 SPI2, J11 GPS, J12 UART1, J13 U.FL_R_SMT, J14 USB_B_Mini, J15 CON-SMA-EDGE-S, J2 Debug, J3 PWR, J4 PWR, J5 IMU, J6 SPI1_IMU, J7 BAR, J8 SPI1_BAR, J9 MAG, SW1 NRST, SW2 BOOT0, SW3 VSEL, U1 STM32F446RCTx, U2 IIS2MDCTR, U3 ATGM336H, U4 LSM6DS3TR-C, U5 LPS25HB, U6 AP2112K-3.3, U7 LMR50410, U9 nRF24L01P, Y1 8MHz, Y2 16MHz

Commit message: Added quadcopter PCB revision 2 and updated README
Parts:
- R6: value R_US -> 1k5
Connections:
- net /Sensors/IIS2_CS renamed /Sensors/MAG_CS
- net /Sensors/IIS2_IRQ renamed /Sensors/MAG_IRQ
- net /Sensors/IIS2_MOSI renamed /Sensors/MAG_MOSI
- net /Sensors/IIS2_SCK renamed /Sensors/MAG_SCK
Changed lines of the file:
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@@
 			(size 0.35 0.3)
 			(layers "F.Cu" "F.Mask" "F.Paste")
-			(net "/Sensors/IIS2_SCK")
+			(net "/Sensors/MAG_SCK")
 			(pinfunction "SCL/SPC_1")
 			(pintype "bidirectional")
@@
 			(size 0.35 0.3)
 			(layers "F.Cu" "F.Mask" "F.Paste")
-			(net "/Sensors/IIS2_CS")
+			(net "/Sensors/MAG_CS")
 			(pinfunction "CS_3")
 			(pintype "input")
@@
 			(size 0.35 0.3)
 			(layers "F.Cu" "F.Mask" "F.Paste")
-			(net "/Sensors/IIS2_IRQ")
+			(net "/Sensors/MAG_IRQ")
 			(pinfunction "INT/DRDY_7")
 			(pintype "output")
@@
 			)
 		)
-		(property "Value" "R_US"
+		(property "Value" "1k5"
 			(at 0 1.65 90)
 			(layer "F.Fab")
@@
 			(layers "F.Cu" "F.Mask" "F.Paste")
 			(roundrect_rratio 0.243902)
-			(net "/Sensors/IIS2_MOSI")
+			(net "/Sensors/MAG_MOSI")
 			(pintype "passive")
 		)
@@
 			(layers "F.Cu" "F.Mask" "F.Paste")
 			(roundrect_rratio 0.25)
-			(net "/Sensors/IIS2_SCK")
+			(net "/Sensors/MAG_SCK")
 			(pinfunction "Pin_1_1")
 			(pintype "passive")
@@
 			(layers "F.Cu" "F.Mask" "F.Paste")
 			(roundrect_rratio 0.25)
-			(net "/Sensors/IIS2_MOSI")
+			(net "/Sensors/MAG_MOSI")
 			(pinfunction "Pin_2_2")
 			(pintype "passive")
@@
 			(layers "F.Cu" "F.Mask" "F.Paste")
 			(roundrect_rratio 0.25)
-			(net "/Sensors/IIS2_CS")
+			(net "/Sensors/MAG_CS")
 			(pinfunction "Pin_3_3")
 			(pintype "passive")
@@
 			(layers "F.Cu" "F.Mask" "F.Paste")
 			(roundrect_rratio 0.25)
-			(net "/Sensors/IIS2_IRQ")
+			(net "/Sensors/MAG_IRQ")
 			(pinfunction "Pin_4_4")
 			(pintype "passive")
@@
 	)
 	(gr_circle
-		(center 99.75 96)
-		(end 100.039736 96)
+		(center 100 98.5)
+		(end 100.289736 98.5)
 		(stroke
 			(width 0.1)
@@
 	)
 	(segment
-		(start 82.075 116.575)
-		(end 82.075 115.25)
-		(width 0.3)
-		(layer "F.Cu")
-		(net "/Sensors/IIS2_SCK")
-	)
-	(segment
-		(start 85.5 120)
-		(end 82.075 116.575)
-		(width 0.3)
-		(layer "F.Cu")
-		(net "/Sensors/IIS2_SCK")
-	)
-	(segment
-		(start 83.25 116)
-		(end 83.075 115.825)
-		(width 0.3)
-		(layer "F.Cu")
-		(net "/Sensors/IIS2_CS")
-	)
-	(segment
-		(start 83.075 115.825)
-		(end 83.075 115.25)
-		(width 0.3)
-		(layer "F.Cu")
-		(net "/Sensors/IIS2_CS")
-	)
-	(segment
-		(start 87.5 120)
-		(end 87.5 118.75)
-		(width 0.3)
-		(layer "F.Cu")
-		(net "/Sensors/IIS2_CS")
-	)
-	(via
-		(at 83.25 116)
-		(size 0.7)
-		(drill 0.3)
-		(layers "F.Cu" "B.Cu")
-		(net "/Sensors/IIS2_CS")
-	)
-	(via
-		(at 87.5 118.75)
-		(size 0.7)
-		(drill 0.3)
-		(layers "F.Cu" "B.Cu")
-		(net "/Sensors/IIS2_CS")
-	)
-	(segment
-		(start 86 118.75)
-		(end 83.25 116)
-		(width 0.3)
-		(layer "B.Cu")
-		(net "/Sensors/IIS2_CS")
-	)
-	(segment
-		(start 87.5 118.75)
-		(end 86 118.75)
-		(width 0.3)
-		(layer "B.Cu")
-		(net "/Sensors/IIS2_CS")
-	)
-	(segment
 		(start 85.175 116.85)
 		(end 83.575 115.25)
@@
 	)
 	(segment
-		(start 83.575 113.175)
-		(end 83.75 113)
-		(width 0.3)
-		(layer "F.Cu")
-		(net "/Sensors/IIS2_IRQ")
-	)
-	(segment
-		(start 88.5 120)
-		(end 88.5 118.75)
-		(width 0.3)
-		(layer "F.Cu")
-		(net "/Sensors/IIS2_IRQ")
-	)
-	(segment
-		(start 83.575 113.75)
-		(end 83.575 113.175)
-		(width 0.3)
-		(layer "F.Cu")
-		(net "/Sensors/IIS2_IRQ")
-	)
-	(via
-		(at 88.5 118.75)
-		(size 0.7)
-		(drill 0.3)
-		(layers "F.Cu" "B.Cu")
-		(net "/Sensors/IIS2_IRQ")
-	)
-	(via
-		(at 83.75 113)
-		(size 0.7)
-		(drill 0.3)
-		(layers "F.Cu" "B.Cu")
-		(net "/Sensors/IIS2_IRQ")
-	)
-	(segment
-		(start 88.5 117.5)
-		(end 84 113)
-		(width 0.3)
-		(layer "B.Cu")
-		(net "/Sensors/IIS2_IRQ")
-	)
-	(segment
-		(start 84 113)
-		(end 83.75 113)
-		(width 0.3)
-		(layer "B.Cu")
-		(net "/Sensors/IIS2_IRQ")
-	)
-	(segment
-		(start 88.5 118.75)
-		(end 88.5 117.5)
-		(width 0.3)
-		(layer "B.Cu")
-		(net "/Sensors/IIS2_IRQ")
-	)
-	(segment
 		(start 102.025 111.8125)
 		(end 102 111.8375)
@@
 	)
 	(segment
-		(start 87 117.25)
-		(end 86.5 117.75)
-		(width 0.3)
-		(layer "F.Cu")
-		(net "/Sensors/IIS2_MOSI")
-	)
-	(segment
-		(start 86.5 117.75)
-		(end 86.5 120)
-		(width 0.3)
-		(layer "F.Cu")
-		(net "/Sensors/IIS2_MOSI")
-	)
-	(segment
 		(start 147.428932 88.476432)
 		(end 148.441432 89.488932)
@@
 		(net "Net-(U7-FB)")
 	)
+	(segment
+		(start 87 117.25)
+		(end 86.5 117.75)
+		(width 0.3)
+		(layer "F.Cu")
+		(net "/Sensors/MAG_MOSI")
+	)
+	(segment
+		(start 86.5 117.75)
+		(end 86.5 120)
+		(width 0.3)
+		(layer "F.Cu")
+		(net "/Sensors/MAG_MOSI")
+	)
+	(segment
+		(start 83.25 116)
+		(end 83.075 115.825)
+		(width 0.3)
+		(layer "F.Cu")
+		(net "/Sensors/MAG_CS")
+	)
+	(segment
+		(start 83.075 115.825)
+		(end 83.075 115.25)
+		(width 0.3)
+		(layer "F.Cu")
+		(net "/Sensors/MAG_CS")
+	)
+	(segment
+		(start 87.5 120)
+		(end 87.5 118.75)
+		(width 0.3)
+		(layer "F.Cu")
+		(net "/Sensors/MAG_CS")
+	)
+	(via
+		(at 83.25 116)
+		(size 0.7)
+		(drill 0.3)
+		(layers "F.Cu" "B.Cu")
+		(net "/Sensors/MAG_CS")
+	)
+	(via
+		(at 87.5 118.75)
+		(size 0.7)
+		(drill 0.3)
+		(layers "F.Cu" "B.Cu")
+		(net "/Sensors/MAG_CS")
+	)
+	(segment
+		(start 86 118.75)
+		(end 83.25 116)
+		(width 0.3)
+		(layer "B.Cu")
+		(net "/Sensors/MAG_CS")
+	)
+	(segment
+		(start 87.5 118.75)
+		(end 86 118.75)
+		(width 0.3)
+		(layer "B.Cu")
+		(net "/Sensors/MAG_CS")
+	)
+	(segment
+		(start 82.075 116.575)
+		(end 82.075 115.25)
+		(width 0.3)
+		(layer "F.Cu")
+		(net "/Sensors/MAG_SCK")
+	)
+	(segment
+		(start 85.5 120)
+		(end 82.075 116.575)
+		(width 0.3)
+		(layer "F.Cu")
+		(net "/Sensors/MAG_SCK")
+	)
+	(segment
+		(start 83.575 113.175)
+		(end 83.75 113)
+		(width 0.3)
+		(layer "F.Cu")
+		(net "/Sensors/MAG_IRQ")
+	)
+	(segment
+		(start 88.5 120)
+		(end 88.5 118.75)
+		(width 0.3)
+		(layer "F.Cu")
+		(net "/Sensors/MAG_IRQ")
+	)
+	(segment
+		(start 83.575 113.75)
+		(end 83.575 113.175)
+		(width 0.3)
+		(layer "F.Cu")
+		(net "/Sensors/MAG_IRQ")
+	)
+	(via
+		(at 88.5 118.75)
+		(size 0.7)
+		(drill 0.3)
+		(layers "F.Cu" "B.Cu")
+		(net "/Sensors/MAG_IRQ")
+	)
+	(via
+		(at 83.75 113)
+		(size 0.7)
+		(drill 0.3)
+		(layers "F.Cu" "B.Cu")
+		(net "/Sensors/MAG_IRQ")
+	)
+	(segment
+		(start 88.5 117.5)
+		(end 84 113)
+		(width 0.3)
+		(layer "B.Cu")
+		(net "/Sensors/MAG_IRQ")
+	)
+	(segment
+		(start 84 113)
+		(end 83.75 113)
+		(width 0.3)
+		(layer "B.Cu")
+		(net "/Sensors/MAG_IRQ")
+	)
+	(segment
+		(start 88.5 118.75)
+		(end 88.5 117.5)
+		(width 0.3)
+		(layer "B.Cu")
+		(net "/Sensors/MAG_IRQ")
+	)
 	(zone
