File: hardware/no_fly_zone/rev1.0/no_fly_zone.kicad_sch (KiCad schematic)
At the start: 12 parts, among them J1 ESC, J10 SPI2, J11 GPS, J12 UART1, J2 Debug, J3 PWR, J4 PWR, J5 IMU, J6 SPI1_IMU, J7 BAR, J8 SPI1_BAR, J9 MAG

Commit message: Added quadcopter PCB revision 2 and updated README
Connections:
- net MCU/IIS2_IRQ renamed MCU/MAG_IRQ
- net Sensors/IIS2_CS renamed Sensors/MAG_CS
- net Sensors/IIS2_IRQ renamed Sensors/MAG_IRQ
- net Sensors/IIS2_MOSI renamed Sensors/MAG_MOSI
- net Sensors/IIS2_SCK renamed Sensors/MAG_SCK
Other:
- sheet MCU ports: added MAG_IRQ, TIM5_CH2, TIM5_CH3; removed IIS2_IRQ, TIM2_CH2, TIM2_CH3
- sheet Sensors ports: added MAG_CS, MAG_IRQ, MAG_MOSI, MAG_SCK; removed IIS2_CS, IIS2_IRQ, IIS2_MOSI, IIS2_SCK
Changed lines of the file:
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@@
-			)
-		)
-		(pin "IIS2_IRQ" input
-			(at 85.09 116.84 0)
-			(effects
-				(font
-					(size 1.27 1.27)
-				)
-				(justify right)
-			)
-		)
-		(pin "IIS2_CS" input
-			(at 85.09 114.3 0)
-			(effects
-				(font
-					(size 1.27 1.27)
-				)
-				(justify right)
-			)
-		)
-		(pin "IIS2_SCK" input
-			(at 85.09 109.22 0)
-			(effects
-				(font
-					(size 1.27 1.27)
-				)
-				(justify right)
-			)
-		)
-		(pin "IIS2_MOSI" input
-			(at 85.09 111.76 0)
-			(effects
-				(font
-					(size 1.27 1.27)
-				)
-				(justify right)
 			)
 		)
@@
 		(pin "+3V3" input
 			(at 85.09 68.58 0)
+			(effects
+				(font
+					(size 1.27 1.27)
+				)
+				(justify right)
+			)
+		)
+		(pin "MAG_IRQ" input
+			(at 85.09 116.84 0)
+			(effects
+				(font
+					(size 1.27 1.27)
+				)
+				(justify right)
+			)
+		)
+		(pin "MAG_MOSI" input
+			(at 85.09 111.76 0)
+			(effects
+				(font
+					(size 1.27 1.27)
+				)
+				(justify right)
+			)
+		)
+		(pin "MAG_SCK" input
+			(at 85.09 109.22 0)
+			(effects
+				(font
+					(size 1.27 1.27)
+				)
+				(justify right)
+			)
+		)
+		(pin "MAG_CS" input
+			(at 85.09 114.3 0)
 			(effects
 				(font
@@
 			)
 		)
-		(pin "TIM2_CH3" input
-			(at 144.78 54.61 180)
-			(effects
-				(font
-					(size 1.27 1.27)
-				)
-				(justify left)
-			)
-		)
 		(pin "TIM2_CH1" input
 			(at 144.78 59.69 180)
@@
 			)
 		)
-		(pin "TIM2_CH2" input
-			(at 144.78 57.15 180)
-			(effects
-				(font
-					(size 1.27 1.27)
-				)
-				(justify left)
-			)
-		)
 		(pin "IMU_IRQ2" input
 			(at 144.78 88.9 180)
@@
 			)
 		)
-		(pin "IIS2_IRQ" input
-			(at 144.78 116.84 180)
-			(effects
-				(font
-					(size 1.27 1.27)
-				)
-				(justify left)
-			)
-		)
 		(pin "IMU_IRQ1" input
 			(at 144.78 86.36 180)
@@
 			(effects
 				(font
+					(size 1.27 1.27)
+				)
+				(justify left)
+			)
+		)
+		(pin "MAG_IRQ" input
+			(at 144.78 116.84 180)
+			(effects
+				(font
+					(size 1.27 1.27)
+				)
+				(justify left)
+			)
+		)
+		(pin "TIM5_CH2" input
+			(at 144.78 54.61 180)
+			(effects
+				(font
+					(size 1.27 1.27)
+				)
+				(justify left)
+			)
+		)
+		(pin "TIM5_CH3" input
+			(at 144.78 57.15 180)
+			(effects
+				(font
