File: hardware/no_fly_zone/rev1.0/sensors.kicad_sch (KiCad schematic)
At the start: 17 parts, among them J13 U.FL_R_SMT, U2 IIS2MDCTR, U3 ATGM336H, U4 LSM6DS3TR-C, U5 LPS25HB

Commit message: Added quadcopter PCB revision 2 and updated README
Connections:
- net IIS2_CS renamed MAG_CS
- net IIS2_IRQ renamed MAG_IRQ
- net IIS2_MOSI renamed MAG_MOSI
- net IIS2_SCK renamed MAG_SCK
Changed lines of the file:
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@@
 		)
 	)
-	(hierarchical_label "IIS2_CS"
+	(hierarchical_label "MAG_CS"
 		(shape input)
 		(at 175.26 54.61 180)
@@
 		)
 	)
-	(hierarchical_label "IIS2_IRQ"
+	(hierarchical_label "MAG_IRQ"
 		(shape input)
 		(at 224.79 57.15 0)
@@
 		)
 	)
-	(hierarchical_label "IIS2_MOSI"
+	(hierarchical_label "MAG_MOSI"
 		(shape input)
 		(at 156.21 49.53 180)
@@
 		)
 	)
-	(hierarchical_label "IIS2_SCK"
+	(hierarchical_label "MAG_SCK"
 		(shape input)
 		(at 175.26 45.72 180)
